File: hw/SummerCart64.sch (EAGLE design)
At the start: 85 parts, among them J1 N64_EDGE, J2 MICRO_SD, J3 MICRO_USB, J4 SSW-106-02-G-D, U1 10M08SCE144C8G, U10 LD117AS33TR, U2 MT48LC16M16A2, U3 ATTINY45, U4 W25Q128JVSIM, U5 IS62WVS2568GBLL-45NLI, U6 93C66, U7 74ABT125PW, U8 MCP7940N, U9 FT2232HL, X1 XLH336, X2 FC-12M, X3 XLH336

Commit message: [SC64][FW][HW][SW] Completely new concept for firmware, abandoned SummerBanger64 for N64-UNFLoader, added UltraCIC-III as submodule, CI configuration
Parts:
- C1, C23: value (none) -> 10n
- C10, C11, C12, C13, C14, C15, C18, C19, C2, C25, C27, C29, C3, C30, C31, C32, C33, C34, C35, C36, C4, C5, C6, C8, C9: value (none) -> 100n
- C16, C17, C26, C28, C37, C38: value (none) -> 4.7u
- C20, C21: value (none) -> 9p
- C22, C7: value (none) -> 47u
- C24: value (none) -> 3.3u
- D1, D2: value BAT60J -> BAT60AE6327HTSA1
- J2: value MICRO_SD -> molex 104031-0811
- J3: value MICRO_USB -> 10118192-0002LF
- L1, L2: value (none) -> MI0603K300R-10
- LD1: value (none) -> 150060RS75000
- R10, R11: value 10K -> 2.2k
- R12, R14: value 10K -> 1k
- R13: value 10K -> 12k
- R9: value 10K -> 10k
- RN1, RN2, RN3, RN4, RN5, RN6, RN7: value (none) -> 47R
- RN10, RN8, RN9: value (none) -> 20k
- S1: value 218-2 -> 218-2LPSTRF
- U10: value LD117AS33TR -> AZ1117IH-3.3TRG1
- U2: value MT48LC16M16A2 -> IS42S16320F-7TL
- U3: value ATTINY45 -> ATTINY45-20XU
- U6: value 93C66 -> AT93C66B-XHM
- U7: value 74ABT125PW -> SN74LVC125APWR
- U8: value MCP7940N -> MCP7940NT-I/ST
- X1: value XLH336 -> XLH336050.000000I
- X2: value FC-12M -> FC-12M 32.7680KA-AC3
- X3: value XLH336 -> XLH336012.000000X
Other:
- note added: "CIC"
- note added: "Crystal Oscillators"
- note added: "FLASH"
- note added: "FPGA"
- note added: "FTDI"
- note added: "FTDI <-> CIC Buffer"
- note added: "FTDI EEPROM"
- note added: "LED"
- note added: "N64 <-> FPGA Resistors"
- note added: "N64 Edge Connector"
- note added: "PMOD"
- note added: "Pull-up Resistors"
- note added: "RTC"
- note added: "SD Card"
- note added: "SDRAM"
- note added: "SRAM"
- moved on the sheet: C1, C10, C11, C12, C13, C14, C15, C16, C17, C18, C19, C2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
