File: hw/v1/SummerCart64.brd (EAGLE design)
At the start: 101.8 x 57.5 mm, 85 parts, among them J1 N64_EDGE, J2 molex 104031-0811, J3 10118192-0002LF, J4 SSW-106-02-G-D, U1 10M08SCE144C8G, U10 AZ1117IH-3.3TRG1, U2 IS42S16320F-7TL, U3 ATTINY45-20XU, U4 W25Q128JVSIM, U5 IS62WVS2568GBLL-45NLI, U6 AT93C66B-XHM, U7 SN74LVC125APWR, U8 MCP7940NT-I/ST, U9 FT2232HL, X1 XLH336050.000000I, X2 FC-12M 32.7680KA-AC3, X3 XLH336012.000000X

Commit message: device_arbiter overhaul, ddipl stuff added
Connections:
- net JTCK_C renamed /INT_C
Changed lines of the file:
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@@
 <wire x1="-5.8" y1="2" x2="-3.1" y2="4.7" width="0.127" layer="1"/>
-</signal>
-<signal name="JTCK_C">
-<contactref element="J1" pad="44"/>
-<contactref element="RN2" pad="1"/>
-<wire x1="-15" y1="-6" x2="-15" y2="0.7" width="0.127" layer="1"/>
-<wire x1="-7.3" y1="2.9" x2="-5.5" y2="4.7" width="0.127" layer="1"/>
-<wire x1="-5.5" y1="4.7" x2="-5.5" y2="5.325" width="0.127" layer="1"/>
-<wire x1="-15" y1="0.7" x2="-12.8" y2="2.9" width="0.127" layer="1"/>
-<wire x1="-12.8" y1="2.9" x2="-7.3" y2="2.9" width="0.127" layer="1"/>
 </signal>
 <signal name="CLK_SDRAM">
@@
 <wire x1="-42.355" y1="24.8" x2="-42.365" y2="24.81" width="0.127" layer="1"/>
 </signal>
+<signal name="/INT_C">
+<contactref element="J1" pad="44"/>
+<contactref element="RN2" pad="1"/>
+<wire x1="-7.3" y1="2.9" x2="-5.5" y2="4.7" width="0.127" layer="1"/>
+<wire x1="-5.5" y1="4.7" x2="-5.5" y2="5.325" width="0.127" layer="1"/>
+<wire x1="-15" y1="0.7" x2="-12.8" y2="2.9" width="0.127" layer="1"/>
+<wire x1="-12.8" y1="2.9" x2="-7.3" y2="2.9" width="0.127" layer="1"/>
+<wire x1="-15" y1="-6" x2="-15" y2="0.7" width="0.127" layer="1"/>
+</signal>
 </signals>
